File: auto_watering.kicad_pcb (KiCad board)
At the start: 2 copper layers, 188 x 91.4 mm, 50 parts, among them K1 SRD12VDC, K2 SRD12VDC, K3 SRD12VDC, K4 SRD12VDC, K5 SRD12VDC, K6 SRD12VDC, U1 PC817, U2 PC817, U3 PC817, U4 PC817, U5 PC817, U6 PC817, U7 ESP32-DevKitC

Commit message: Remove JLC marking on PCB
Other:
- board text removed: "JLCJLCJLCJLC"
